Commit message: Fix motion tracker teleoperation for calibrated dual FR3
Add serial-based tracker input and diagnostics, enforce tracker freshness and motion limits, synchronize the calibrated MuJoCo and Pinocchio models, simplify runtime commands, and make joint-space reset duration obey explicit speed and acceleration bounds.

File: teleop_sources/pico/assets/dual_fr3/dual_fr3_kinematics.urdf (robot description, URDF)
Before this commit: robot mounted_dual_fr3, 19 links, 18 joints
Joints:
- joint left_mount: origin xyz=-0.038 -0.18 0.304 rpy=-0.5567600306 0.5689773370 -2.4626595739 -> xyz=0.013079894 0.100675805 -0.005974552 rpy=-0.78850572 0.02334617 0.01037711
- joint right_mount: origin xyz=-0.038 0.18 0.304 rpy=0.5567600306 0.5689773370 2.4626595739 -> xyz=-0.013079894 -0.100675805 0.005974552 rpy=0.76133216 0.03792674 -0.01038175
