Commit message: Run both O30-family hands on the corrected 0803 limits
The 0706 URDF's joint limits were wrong on all 20 joints; the tick map
anchors on them, which was the whole sim-to-real pinch gap. All pinned
copies (assets URDF, driver contract, bridge and teleop_data profiles)
move to 0803 together; the guard tests keep them locked.

The left mount is an O30 now, not a G20: the o30i node, bridge profile,
launch and both compose files go side-generic (per-side CANFD device
index, left=0 right=1), every teleop entry point defaults to dual o30i,
and identify_canfd_devices probes both request IDs -- it used to ask
with the right hand's ID only and report a healthy left hand as
silence. Test scripts gain --side and park at URDF-0-deg neutral
computed from the contract, because all-ticks-0 splays the yaws onto
the index's pinched cable.

Known left residual: the metal tips miss laterally at a model-verified
contact pose -- likely the O30-vs-O30i URDF difference; vendor asked.

Co-Authored-By: Claude Fable 5 <noreply@anthropic.com>

File: assets/linkerhand_o30i/right/linkerhand_o30i_right.urdf (robot description, URDF)
Before this commit: robot linkerhand_O30i_right.urdf, 21 links, 20 joints
Joints:
- joint index_dip: limit lower=0 upper=1.66112 effort=1 velocity=1 -> lower=0.0 upper=1.5016 effort=1 velocity=1
- joint index_mcp_pitch: limit lower=0 upper=1.72918 effort=1 velocity=1 -> lower=0.0 upper=1.5050 effort=1 velocity=1
- joint index_mcp_roll: limit lower=-0.4 upper=0.03711 effort=1 velocity=1 -> lower=-0.3741 upper=0.03711 effort=1 velocity=1
- joint index_pip: limit lower=0 upper=1.63 effort=1 velocity=1 -> lower=0.0 upper=1.5765 effort=1 velocity=1
- joint middle_dip: limit lower=0 upper=1.5863 effort=1 velocity=1 -> lower=0.0 upper=1.5207 effort=1 velocity=1
- joint middle_mcp_pitch: limit lower=0 upper=1.884 effort=1 velocity=1 -> lower=0.0 upper=1.6159 effort=1 velocity=1
- joint middle_mcp_roll: limit lower=-0.38 upper=0.05418 effort=1 velocity=1 -> lower=-0.4906 upper=0.05418 effort=1 velocity=1
- joint middle_pip: limit lower=0 upper=1.7071 effort=1 velocity=1 -> lower=0.0 upper=1.5783 effort=1 velocity=1
- joint pinky_dip: limit lower=0 upper=1.7331 effort=1 velocity=1 -> lower=0.0 upper=1.5549 effort=1 velocity=1
- joint pinky_mcp_pitch: limit lower=0 upper=1.8497 effort=1 velocity=1 -> lower=0.0 upper=1.6152 effort=1 velocity=1
- joint pinky_mcp_roll: limit lower=-0.28 upper=0.28103 effort=1 velocity=1 -> lower=-0.1835 upper=0.2810 effort=1 velocity=1
- joint pinky_pip: limit lower=0 upper=1.7026 effort=1 velocity=1 -> lower=0.0 upper=1.4858 effort=1 velocity=1
- joint ring_dip: limit lower=0 upper=1.6749 effort=1 velocity=1 -> lower=0.0 upper=1.4986 effort=1 velocity=1
- joint ring_mcp_pitch: limit lower=0 upper=1.9626 effort=1 velocity=1 -> lower=0.0 upper=1.6596 effort=1 velocity=1
- joint ring_mcp_roll: limit lower=-0.28 upper=0.18823 effort=0 velocity=0 -> lower=-0.1371 upper=0.18823 effort=0 velocity=0
- joint ring_pip: limit lower=0 upper=1.6621 effort=1 velocity=1 -> lower=0.0 upper=1.5009 effort=1 velocity=1
- joint thumb_cmc_roll: limit lower=0 upper=0.6108 effort=1 velocity=1 -> lower=0.0 upper=0.5731 effort=1 velocity=1
- joint thumb_cmc_yaw: limit lower=0 upper=2.094 effort=1 velocity=1 -> lower=0.0 upper=1.9268 effort=1 velocity=1
- joint thumb_ip: limit lower=0 upper=1.733 effort=1 velocity=1 -> lower=0.0 upper=1.5910 effort=1 velocity=1
- joint thumb_mcp: limit lower=0 upper=1.7134 effort=1 velocity=1 -> lower=0.0 upper=1.5194 effort=1 velocity=1
